Commit message: Modified the joint limits of Gen3 and Gen3 Lite robots as per the values in the User Guides (#241)

File: kortex_description/arms/gen3/6dof/urdf/gen3_macro.xacro (robot description, xacro)
@@ -174,5 +174,5 @@
       <child link="${prefix}bicep_link" />
       <axis xyz="0 0 1" />
-      <limit lower="-2.41" upper="2.41" effort="39" velocity="1.3963" />
+      <limit lower="-2.24" upper="2.24" effort="39" velocity="1.3963" />
     </joint>
     <link name="${prefix}forearm_link">
@@ -203,5 +203,5 @@
       <child link="${prefix}forearm_link" />
       <axis xyz="0 0 1" />
-      <limit lower="-2.66" upper="2.66" effort="39" velocity="1.3963" />
+      <limit lower="-2.57" upper="2.57" effort="39" velocity="1.3963" />
     </joint>
     <link name="${prefix}spherical_wrist_1_link">
@@ -272,5 +272,5 @@
       <child link="${prefix}spherical_wrist_2_link" />
       <axis xyz="0 0 1" />
-      <limit lower="-2.23" upper="2.23" effort="9" velocity="1.2218" />
+      <limit lower="-2.09" upper="2.09" effort="9" velocity="1.2218" />
     </joint>
     <xacro:if value="${vision}">

File: kortex_description/arms/gen3/7dof/urdf/gen3_macro.xacro (robot description, xacro)
@@ -173,5 +173,5 @@
       <axis
         xyz="0 0 1" />
-      <limit lower="-2.41" upper="2.41" effort="39" velocity="1.3963" />
+      <limit lower="-2.24" upper="2.24" effort="39" velocity="1.3963" />
     </joint>
     <link name="half_arm_2_link${prefix}">
@@ -263,5 +263,5 @@
       <axis
         xyz="0 0 1" />
-      <limit lower="-2.66" upper="2.66" effort="39" velocity="1.3963" />
+      <limit lower="-2.57" upper="2.57" effort="39" velocity="1.3963" />
     </joint>
     <link name="spherical_wrist_1_link${prefix}">
@@ -353,5 +353,5 @@
       <axis
         xyz="0 0 1" />
-      <limit lower="-2.23" upper="2.23" effort="9" velocity="1.2218" />
+      <limit lower="-2.09" upper="2.09" effort="9" velocity="1.2218" />
     </joint>
     <xacro:if value="${vision}">

File: kortex_description/arms/gen3_lite/6dof/urdf/gen3_lite_macro.xacro (robot description, xacro)
@@ -122,5 +122,5 @@
       <child link="${prefix}shoulder_link" />
       <axis xyz="0 0 1" />
-      <limit lower="-2.69" upper="2.69" effort="10" velocity="1.6" />
+      <limit lower="-2.68" upper="2.68" effort="10" velocity="1.6" />
     </joint>
     <link name="${prefix}arm_link">
@@ -154,5 +154,5 @@
       <child link="${prefix}arm_link" />
       <axis xyz="0 0 1" />
-      <limit lower="-2.69" upper="2.69" effort="14" velocity="1.6" />
+      <limit lower="-2.61" upper="2.61" effort="14" velocity="1.6" />
     </joint>
     <link name="${prefix}forearm_link">
@@ -186,5 +186,5 @@
       <child link="${prefix}forearm_link" />
       <axis xyz="0 0 1" />
-      <limit lower="-2.69" upper="2.69" effort="10" velocity="1.6" />
+      <limit lower="-2.61" upper="2.61" effort="10" velocity="1.6" />
     </joint>
     <link name="${prefix}lower_wrist_link">
@@ -218,5 +218,5 @@
       <child link="${prefix}lower_wrist_link" />
       <axis xyz="0 0 1" />
-      <limit lower="-2.59" upper="2.59" effort="7" velocity="1.6" />
+      <limit lower="-2.6" upper="2.6" effort="7" velocity="1.6" />
     </joint>
     <link name="${prefix}upper_wrist_link">
@@ -250,5 +250,5 @@
       <child link="${prefix}upper_wrist_link" />
       <axis xyz="0 0 1" />
-      <limit lower="-2.57" upper="2.57" effort="7" velocity="1.6" />
+      <limit lower="-2.53" upper="2.53" effort="7" velocity="1.6" />
     </joint>
     <link name="${prefix}end_effector_link"/>
@@ -258,5 +258,5 @@
       <child link="${prefix}end_effector_link" />
       <axis xyz="0 0 1" />
-      <limit lower="-2.59" upper="2.59" effort="7" velocity="3.2" />
+      <limit lower="-2.6" upper="2.6" effort="7" velocity="3.2" />
     </joint>
     <link name="${prefix}dummy_link" />
