Commit message: moving prefix and making control tag optional

File: kortex_description/arms/gen3/7dof/urdf/gen3_macro.xacro (robot description, xacro)
@@ -26,38 +26,42 @@
     sim_ignition:=false
     sim_isaac:=false
+    use_kortex_control:=false
     isaac_joint_commands:=/isaac_joint_commands
     isaac_joint_states:=/isaac_joint_states
     use_external_cable:=false
     initial_positions:=${dict(joint_1=0.0,joint_2=0.0,joint_3=0.0,joint_4=0.0,joint_5=0.0,joint_6=0.0,joint_7=0.0)}" >
-    <!-- ros2 control include -->
-    <xacro:include filename="$(find kortex_description)/arms/gen3/${dof}dof/urdf/kortex.ros2_control.xacro" />
-    <xacro:kortex_ros2_control
-      name="${prefix}KortexMultiInterfaceHardware" prefix="${prefix}"
-      use_fake_hardware="${use_fake_hardware}"
-      fake_sensor_commands="${fake_sensor_commands}"
-      sim_gazebo="${sim_gazebo}"
-      sim_ignition="${sim_ignition}"
-      sim_isaac="${sim_isaac}"
-      isaac_joint_commands="${isaac_joint_commands}"
-      isaac_joint_states="${isaac_joint_states}"
-      tf_prefix=""
-      initial_positions="${initial_positions}"
-      robot_ip="${robot_ip}"
-      username="${username}"
-      password="${password}"
-      port="${port}"
-      port_realtime="${port_realtime}"
-      session_inactivity_timeout_ms="${session_inactivity_timeout_ms}"
-      connection_inactivity_timeout_ms="${connection_inactivity_timeout_ms}"
-      use_internal_bus_gripper_comm="${use_internal_bus_gripper_comm}"
-      gripper_max_velocity="${gripper_max_velocity}"
-      gripper_max_force="${gripper_max_force}"
-      gripper_joint_name="${gripper_joint_name}"/>
-    <joint name="${prefix}base_joint" type="fixed">
+    <xacro:if value="${use_kortex_control}">
+      <!-- ros2 control include -->
+      <xacro:include filename="$(find kortex_description)/arms/gen3/${dof}dof/urdf/kortex.ros2_control.xacro" />
+      <xacro:kortex_ros2_control
+        name="${prefix}KortexMultiInterfaceHardware" prefix="${prefix}"
+        use_fake_hardware="${use_fake_hardware}"
+        use_kortex_control="${use_kortex_control}"
+        fake_sensor_commands="${fake_sensor_commands}"
+        sim_gazebo="${sim_gazebo}"
+        sim_ignition="${sim_ignition}"
+        sim_isaac="${sim_isaac}"
+        isaac_joint_commands="${isaac_joint_commands}"
+        isaac_joint_states="${isaac_joint_states}"
+        tf_prefix=""
+        initial_positions="${initial_positions}"
+        robot_ip="${robot_ip}"
+        username="${username}"
+        password="${password}"
+        port="${port}"
+        port_realtime="${port_realtime}"
+        session_inactivity_timeout_ms="${session_inactivity_timeout_ms}"
+        connection_inactivity_timeout_ms="${connection_inactivity_timeout_ms}"
+        use_internal_bus_gripper_comm="${use_internal_bus_gripper_comm}"
+        gripper_max_velocity="${gripper_max_velocity}"
+        gripper_max_force="${gripper_max_force}"
+        gripper_joint_name="${gripper_joint_name}"/>
+    </xacro:if>
+    <joint name="base_joint${prefix}" type="fixed">
       <xacro:insert_block name="origin" />
       <parent link="${parent}"/>
-      <child link="${prefix}base_link" />
+      <child link="base_link${prefix}" />
     </joint>
-    <link name="${prefix}base_link">
+    <link name="base_link${prefix}">
       <inertial>
         <origin xyz="-0.000648 -0.000166 0.084487" rpy="0 0 0" />
@@ -81,5 +85,5 @@
       </collision>
     </link>
-    <link name="${prefix}shoulder_link">
+    <link name="shoulder_link${prefix}">
       <inertial>
         <origin xyz="-2.3E-05 -0.010364 -0.07336" rpy="0 0 0" />
@@ -105,11 +109,11 @@
     <xacro:if value="${use_external_cable}">
       <joint
-      name="${prefix}joint_1"
+      name="joint_1${prefix}"
       type="revolute">
         <origin xyz="0 0 0.15643" rpy="3.1416 2.7629E-18 -4.9305E-36" />
         <parent
-          link="${prefix}base_link" />
-        <child
-          link="${prefix}shoulder_link" />
+          link="base_link${prefix}" />
+        <child
+          link="shoulder_link${prefix}" />
         <axis
           xyz="0 0 1" />
@@ -123,11 +127,11 @@
     <xacro:unless value="${use_external_cable}">
       <joint
-        name="${prefix}joint_1"
+        name="joint_1${prefix}"
         type="continuous">
         <origin xyz="0 0 0.15643" rpy="3.1416 2.7629E-18 -4.9305E-36" />
         <parent
-          link="${prefix}base_link" />
-        <child
-          link="${prefix}shoulder_link" />
+          link="base_link${prefix}" />
+        <child
+          link="shoulder_link${prefix}" />
         <axis
           xyz="0 0 1" />
@@ -137,5 +141,5 @@
       </joint>
     </xacro:unless>
-    <link name="${prefix}half_arm_1_link">
+    <link name="half_arm_1_link${prefix}">
       <inertial>
         <origin xyz="-4.4E-05 -0.09958 -0.013278" rpy="0 0 0" />
@@ -160,16 +164,16 @@
     </link>
     <joint
-      name="${prefix}joint_2"
+      name="joint_2${prefix}"
       type="revolute">
       <origin xyz="0 0.005375 -0.12838" rpy="1.5708 2.1343E-17 -1.1102E-16" />
       <parent
-        link="${prefix}shoulder_link" />
+        link="shoulder_link${prefix}" />
       <child
-        link="${prefix}half_arm_1_link" />
+        link="half_arm_1_link${prefix}" />
       <axis
         xyz="0 0 1" />
       <limit lower="-2.41" upper="2.41" effort="39" velocity="1.3963" />
     </joint>
-    <link name="${prefix}half_arm_2_link">
+    <link name="half_arm_2_link${prefix}">
       <inertial>
         <origin xyz="-4.4E-05 -0.006641 -0.117892" rpy="0 0 0" />
@@ -195,11 +199,11 @@
     <xacro:if value="${use_external_cable}">
       <joint
-        name="${prefix}joint_3"
+        name="joint_3${prefix}"
         type="revolute">
         <origin xyz="0 -0.21038 -0.006375" rpy="-1.5708 1.2326E-32 -2.9122E-16" />
         <parent
-          link="${prefix}half_arm_1_link" />
-        <child
-          link="${prefix}half_arm_2_link" />
+          link="half_arm_1_link${prefix}" />
+        <child
+          link="half_arm_2_link${prefix}" />
         <axis
           xyz="0 0 1" />
@@ -213,11 +217,11 @@
     <xacro:unless value="${use_external_cable}">
       <joint
-        name="${prefix}joint_3"
+        name="joint_3${prefix}"
         type="continuous">
         <origin xyz="0 -0.21038 -0.006375" rpy="-1.5708 1.2326E-32 -2.9122E-16" />
         <parent
-          link="${prefix}half_arm_1_link" />
-        <child
-          link="${prefix}half_arm_2_link" />
+          link="half_arm_1_link${prefix}" />
+        <child
+          link="half_arm_2_link${prefix}" />
         <axis
           xyz="0 0 1" />
@@ -227,5 +231,5 @@
       </joint>
     </xacro:unless>
-    <link name="${prefix}forearm_link">
+    <link name="forearm_link${prefix}">
       <inertial>
         <origin xyz="-1.8E-05 -0.075478 -0.015006" rpy="0 0 0" />
@@ -250,16 +254,16 @@
     </link>
     <joint
-      name="${prefix}joint_4"
+      name="joint_4${prefix}"
       type="revolute">
       <origin xyz="0 0.006375 -0.21038" rpy="1.5708 -6.6954E-17 -1.6653E-16" />
       <parent
-        link="${prefix}half_arm_2_link" />
+        link="half_arm_2_link${prefix}" />
       <child
-        link="${prefix}forearm_link" />
+        link="forearm_link${prefix}" />
       <axis
         xyz="0 0 1" />
       <limit lower="-2.66" upper="2.66" effort="39" velocity="1.3963" />
     </joint>
-    <link name="${prefix}spherical_wrist_1_link">
+    <link name="spherical_wrist_1_link${prefix}">
       <inertial>
         <origin xyz="1E-06 -0.009432 -0.063883" rpy="0 0 0" />
@@ -285,11 +289,11 @@
     <xacro:if value="${use_external_cable}">
       <joint
-        name="${prefix}joint_5"
+        name="joint_5${prefix}"
         type="revolute">
         <origin xyz="0 -0.20843 -0.006375" rpy="-1.5708 2.2204E-16 -6.373E-17" />
         <parent
-          link="${prefix}forearm_link" />
-        <child
-          link="${prefix}spherical_wrist_1_link" />
+          link="forearm_link${prefix}" />
+        <child
+          link="spherical_wrist_1_link${prefix}" />
         <axis
           xyz="0 0 1" />
@@ -303,11 +307,11 @@
     <xacro:unless value="${use_external_cable}">
       <joint
-        name="${prefix}joint_5"
+        name="joint_5${prefix}"
         type="continuous">
         <origin xyz="0 -0.20843 -0.006375" rpy="-1.5708 2.2204E-16 -6.373E-17" />
         <parent
-          link="${prefix}forearm_link" />
-        <child
-          link="${prefix}spherical_wrist_1_link" />
+          link="forearm_link${prefix}" />
+        <child
+          link="spherical_wrist_1_link${prefix}" />
         <axis
           xyz="0 0 1" />
@@ -317,5 +321,5 @@
       </joint>
     </xacro:unless>
-    <link name="${prefix}spherical_wrist_2_link">
+    <link name="spherical_wrist_2_link${prefix}">
       <inertial>
         <origin xyz="1E-06 -0.045483 -0.00965" rpy="0 0 0" />
@@ -340,11 +344,11 @@
     </link>
     <joint
-      name="${prefix}joint_6"
+      name="joint_6${prefix}"
       type="revolute">
       <origin xyz="0 0.00017505 -0.10593" rpy="1.5708 9.2076E-28 -8.2157E-15" />
       <parent
-        link="${prefix}spherical_wrist_1_link" />
+        link="spherical_wrist_1_link${prefix}" />
       <child
-        link="${prefix}spherical_wrist_2_link" />
+        link="spherical_wrist_2_link${prefix}" />
       <axis
         xyz="0 0 1" />
@@ -352,5 +356,5 @@
     </joint>
     <xacro:if value="${vision}">
-    <link name="${prefix}bracelet_link">
+    <link name="bracelet_link${prefix}">
       <inertial>
         <origin xyz="0.000281 0.011402 -0.029798" rpy="0 0 0" />
@@ -376,5 +380,5 @@
     </xacro:if>
     <xacro:unless value="${vision}">
-    <link name="${prefix}bracelet_link">
+    <link name="bracelet_link${prefix}">
       <inertial>
         <origin xyz="-9.3E-05 0.000132 -0.022905" rpy="0 0 0" />
@@ -401,11 +405,11 @@
     <xacro:if value="${use_external_cable}">
       <joint
-        name="${prefix}joint_7"
+        name="joint_7${prefix}"
         type="revolute">
         <origin xyz="0 -0.10593 -0.00017505" rpy="-1.5708 -5.5511E-17 9.6396E-17" />
         <parent
-          link="${prefix}spherical_wrist_2_link" />
-        <child
-          link="${prefix}bracelet_link" />
+          link="spherical_wrist_2_link${prefix}" />
+        <child
+          link="bracelet_link${prefix}" />
         <axis
           xyz="0 0 1" />
@@ -419,11 +423,11 @@
     <xacro:unless value="${use_external_cable}">
       <joint
-        name="${prefix}joint_7"
+        name="joint_7${prefix}"
         type="continuous">
         <origin xyz="0 -0.10593 -0.00017505" rpy="-1.5708 -5.5511E-17 9.6396E-17" />
         <parent
-          link="${prefix}spherical_wrist_2_link" />
-        <child
-          link="${prefix}bracelet_link" />
+          link="spherical_wrist_2_link${prefix}" />
+        <child
+          link="bracelet_link${prefix}" />
         <axis
           xyz="0 0 1" />
@@ -433,13 +437,13 @@
       </joint>
     </xacro:unless>
-    <link name="${prefix}end_effector_link" />
+    <link name="end_effector_link${prefix}" />
     <joint
-      name="${prefix}end_effector"
+      name="end_effector${prefix}"
       type="fixed">
       <origin xyz="0 0 -0.0615250000000001" rpy="3.14159265358979 1.09937075168372E-32 0" />
       <parent
-        link="${prefix}bracelet_link" />
+        link="bracelet_link${prefix}" />
       <child
-        link="${prefix}end_effector_link" />
+        link="end_effector_link${prefix}" />
       <axis
         xyz="0 0 0" />
@@ -448,41 +452,41 @@
       <!-- sim camera needs to be rotated which might not apply to built in vision module -->
       <xacro:if value="${sim_ignition}">
-        <link name="${prefix}camera_link" />
-        <joint name="${prefix}camera_module" type="fixed">
+        <link name="camera_link${prefix}" />
+        <joint name="camera_module${prefix}" type="fixed">
           <origin xyz="0 0.05639 0.01305" rpy="0 ${-PI/2} ${-PI/2}" />
-          <parent link="${prefix}end_effector_link" />
-          <child  link="${prefix}camera_link" />
-        </joint>
-        <link name="${prefix}camera_depth_frame" />
-        <joint name="${prefix}depth_module" type="fixed">
+          <parent link="end_effector_link${prefix}" />
+          <child  link="camera_link${prefix}" />
+        </joint>
+        <link name="camera_depth_frame${prefix}" />
+        <joint name="depth_module${prefix}" type="fixed">
           <origin xyz="0.0275 0.066 0.01305" rpy="0 ${-PI/2} ${-PI/2}" />
-          <parent link="${prefix}end_effector_link" />
-          <child  link="${prefix}camera_depth_frame" />
-        </joint>
-        <link name="${prefix}camera_color_frame" />
-        <joint name="${prefix}color_module" type="fixed">
+          <parent link="end_effector_link${prefix}" />
+          <child  link="camera_depth_frame${prefix}" />
+        </joint>
+        <link name="camera_color_frame${prefix}" />
+        <joint name="color_module${prefix}" type="fixed">
           <origin xyz="0 0.05639 0.01305" rpy="0 ${-PI/2} ${-PI/2}" />
-          <parent link="${prefix}end_effector_link" />
-          <child  link="${prefix}camera_color_frame" />
+          <parent link="end_effector_link${prefix}" />
+          <child  link="camera_color_frame${prefix}" />
         </joint>
       </xacro:if>
       <xacro:unless value="${sim_ignition}">
-        <link name="${prefix}camera_link" />
-        <joint name="${prefix}camera_module" type="fixed">
+        <link name="camera_link${prefix}" />
+        <joint name="camera_module${prefix}" type="fixed">
           <origin xyz="0 0.05639 -0.00305" rpy="${PI} ${PI} 0" />
-          <parent link="${prefix}end_effector_link" />
-          <child  link="${prefix}camera_link" />
-        </joint>
-        <link name="${prefix}camera_depth_frame" />
-        <joint name="${prefix}depth_module" type="fixed">
+          <parent link="end_effector_link${prefix}" />
+          <child  link="camera_link${prefix}" />
+        </joint>
+        <link name="camera_depth_frame${prefix}" />
+        <joint name="depth_module${prefix}" type="fixed">
           <origin xyz="0.0275 0.066 -0.00305" rpy="${PI} ${PI} 0" />
-          <parent link="${prefix}end_effector_link" />
-          <child  link="${prefix}camera_depth_frame" />
-        </joint>
-        <link name="${prefix}camera_color_frame" />
-        <joint name="${prefix}color_module" type="fixed">
+          <parent link="end_effector_link${prefix}" />
+          <child  link="camera_depth_frame${prefix}" />
+        </joint>
+        <link name="camera_color_frame${prefix}" />
+        <joint name="color_module${prefix}" type="fixed">
           <origin xyz="0 0.05639 -0.00305" rpy="${PI} ${PI} 0" />
-          <parent link="${prefix}end_effector_link" />
-          <child  link="${prefix}camera_color_frame" />
+          <parent link="end_effector_link${prefix}" />
+          <child  link="camera_color_frame${prefix}" />
         </joint>
       </xacro:unless>

File: kortex_description/arms/gen3/7dof/urdf/kortex.ros2_control.xacro (robot description, xacro)
@@ -58,5 +58,5 @@
         </xacro:unless>
       </hardware>
-      <joint name="${prefix}joint_1">
+      <joint name="joint_1${prefix}">
         <command_interface name="position">
           <param name="min">{-2*pi}</param>
@@ -69,5 +69,5 @@
         <state_interface name="effort"/>
       </joint>
-      <joint name="${prefix}joint_2">
+      <joint name="joint_2${prefix}">
         <command_interface name="position">
           <param name="min">-2.41</param>
@@ -80,5 +80,5 @@
         <state_interface name="effort"/>
       </joint>
-      <joint name="${prefix}joint_3">
+      <joint name="joint_3${prefix}">
         <command_interface name="position">
           <param name="min">{-2*pi}</param>
@@ -91,5 +91,5 @@
         <state_interface name="effort"/>
       </joint>
-      <joint name="${prefix}joint_4">
+      <joint name="joint_4${prefix}">
         <command_interface name="position">
           <param name="min">-2.66</param>
@@ -102,5 +102,5 @@
         <state_interface name="effort"/>
       </joint>
-      <joint name="${prefix}joint_5">
+      <joint name="joint_5${prefix}">
         <command_interface name="position">
           <param name="min">{-2*pi}</param>
@@ -113,5 +113,5 @@
         <state_interface name="effort"/>
       </joint>
-      <joint name="${prefix}joint_6">
+      <joint name="joint_6${prefix}">
         <command_interface name="position">
           <param name="min">-2.23</param>
@@ -124,5 +124,5 @@
         <state_interface name="effort"/>
       </joint>
-      <joint name="${prefix}joint_7">
+      <joint name="joint_7${prefix}">
         <command_interface name="position">
           <param name="min">{-2*pi}</param>
@@ -137,5 +137,5 @@
       <xacro:unless value="${use_fake_hardware or sim_gazebo or sim_ignition or sim_isaac}">
         <xacro:if value="${use_internal_bus_gripper_comm}">
-          <joint name="${prefix}${gripper_joint_name}">
+          <joint name="${gripper_joint_name}${prefix}">
             <command_interface name="position" />
             <state_interface name="position"/>

File: kortex_description/robots/kortex_robot.xacro (robot description, xacro)
@@ -23,4 +23,5 @@
     sim_ignition:=false
     sim_isaac:=false
+    use_kortex_control:=false
     isaac_joint_commands:=/isaac_joint_commands
     isaac_joint_states:=/isaac_joint_states
@@ -46,4 +47,5 @@
       prefix="${prefix}"
       use_internal_bus_gripper_comm="${use_internal_bus_gripper_comm}"
+      use_kortex_control="${use_kortex_control}"
       use_fake_hardware="${use_fake_hardware}"
       fake_sensor_commands="${fake_sensor_commands}"
@@ -62,9 +64,9 @@
     <!-- If no gripper, define tool frame here -->
     <xacro:if value="${not gripper}">
-      <link name="${prefix}tool_frame"/>
-      <joint name="${prefix}tool_frame_joint" type="fixed">
+      <link name="tool_frame${prefix}"/>
+      <joint name="tool_frame_joint${prefix}" type="fixed">
         <origin xyz="0 0 0" rpy="0 0 0" />
-        <parent link="${prefix}${last_arm_link}" />
-        <child link="${prefix}tool_frame" />
+        <parent link="${last_arm_link}${prefix}" />
+        <child link="tool_frame${prefix}" />
         <axis xyz="0 0 0" />
       </joint>
@@ -75,5 +77,5 @@
       <!-- last_arm_link is defined in "$(find kortex_description)/arms/${arm}/urdf/${arm}_macro.xacro" -->
       <xacro:load_gripper
-        parent="${prefix}${last_arm_link}"
+        parent="${last_arm_link}${prefix}"
         prefix="${prefix}"
         use_fake_hardware="${use_fake_hardware}"
