Commit message: Enable architectural calibration
Address review

File: kortex_description/arms/gen3/7dof/urdf/gen3_macro.xacro (robot description, xacro)
@@ -30,5 +30,15 @@
     isaac_joint_states:=/isaac_joint_states
     use_external_cable:=false
-    initial_positions:=${dict(joint_1=0.0,joint_2=0.0,joint_3=0.0,joint_4=0.0,joint_5=0.0,joint_6=0.0,joint_7=0.0)}" >
+    initial_positions:=${dict(joint_1=0.0,joint_2=0.0,joint_3=0.0,joint_4=0.0,joint_5=0.0,joint_6=0.0,joint_7=0.0)}
+    architectural_calibrations:=${
+    dict(
+      joint_1=dict(x=0, y=0, z=0, roll=0, pitch=0, yaw=0),
+      joint_2=dict(x=0, y=0, z=0, roll=0, pitch=0, yaw=0),
+      joint_3=dict(x=0, y=0, z=0, roll=0, pitch=0, yaw=0),
+      joint_4=dict(x=0, y=0, z=0, roll=0, pitch=0, yaw=0),
+      joint_5=dict(x=0, y=0, z=0, roll=0, pitch=0, yaw=0),
+      joint_6=dict(x=0, y=0, z=0, roll=0, pitch=0, yaw=0),
+      joint_7=dict(x=0, y=0, z=0, roll=0, pitch=0, yaw=0)
+    )}" >
     <xacro:if value="${use_kortex_control}">
       <!-- ros2 control include -->
@@ -111,5 +121,7 @@
       name="joint_1${prefix}"
       type="revolute">
-        <origin xyz="0 0 0.15643" rpy="3.1416 2.7629E-18 -4.9305E-36" />
+        <origin
+          xyz="${architectural_calibrations['joint_1']['x']} ${architectural_calibrations['joint_1']['y']} ${architectural_calibrations['joint_1']['z'] + 0.15643}"
+          rpy="${architectural_calibrations['joint_1']['roll'] + PI} ${architectural_calibrations['joint_1']['pitch']} ${architectural_calibrations['joint_1']['yaw']}" />
         <parent
           link="base_link${prefix}" />
@@ -129,5 +141,6 @@
         name="joint_1${prefix}"
         type="continuous">
-        <origin xyz="0 0 0.15643" rpy="3.1416 2.7629E-18 -4.9305E-36" />
+        <origin xyz="${architectural_calibrations['joint_1']['x']} ${architectural_calibrations['joint_1']['y']} ${architectural_calibrations['joint_1']['z'] + 0.15643}"
+          rpy="${architectural_calibrations['joint_1']['roll'] + PI} ${architectural_calibrations['joint_1']['pitch']} ${architectural_calibrations['joint_1']['yaw']}" />
         <parent
           link="base_link${prefix}" />
@@ -166,5 +179,7 @@
       name="joint_2${prefix}"
       type="revolute">
-      <origin xyz="0 0.005375 -0.12838" rpy="1.5708 2.1343E-17 -1.1102E-16" />
+      <origin
+        xyz="${architectural_calibrations['joint_2']['x']} ${architectural_calibrations['joint_2']['y'] + 0.005375} ${architectural_calibrations['joint_2']['z'] - 0.12838}"
+        rpy="${architectural_calibrations['joint_2']['roll'] + PI/2} ${architectural_calibrations['joint_2']['pitch']} ${architectural_calibrations['joint_2']['yaw']}" />
       <parent
         link="shoulder_link${prefix}" />
@@ -201,5 +216,7 @@
         name="joint_3${prefix}"
         type="revolute">
-        <origin xyz="0 -0.21038 -0.006375" rpy="-1.5708 1.2326E-32 -2.9122E-16" />
+        <origin
+          xyz="${architectural_calibrations['joint_3']['x']} ${architectural_calibrations['joint_3']['y'] - 0.21038} ${architectural_calibrations['joint_3']['z'] - 0.006375}"
+          rpy="${architectural_calibrations['joint_3']['roll'] -PI/2} ${architectural_calibrations['joint_3']['pitch']} ${architectural_calibrations['joint_3']['yaw']}" />
         <parent
           link="half_arm_1_link${prefix}" />
@@ -219,5 +236,7 @@
         name="joint_3${prefix}"
         type="continuous">
-        <origin xyz="0 -0.21038 -0.006375" rpy="-1.5708 1.2326E-32 -2.9122E-16" />
+        <origin
+          xyz="${architectural_calibrations['joint_3']['x']} ${architectural_calibrations['joint_3']['y'] - 0.21038} ${architectural_calibrations['joint_3']['z'] - 0.006375}"
+          rpy="${architectural_calibrations['joint_3']['roll'] - PI/2} ${architectural_calibrations['joint_3']['pitch']} ${architectural_calibrations['joint_3']['yaw']}" />
         <parent
           link="half_arm_1_link${prefix}" />
@@ -256,5 +275,7 @@
       name="joint_4${prefix}"
       type="revolute">
-      <origin xyz="0 0.006375 -0.21038" rpy="1.5708 -6.6954E-17 -1.6653E-16" />
+      <origin
+        xyz="${architectural_calibrations['joint_4']['x']} ${architectural_calibrations['joint_4']['y'] + 0.006375} ${architectural_calibrations['joint_4']['z'] - 0.21038}"
+        rpy="${architectural_calibrations['joint_4']['roll'] + PI/2} ${architectural_calibrations['joint_4']['pitch']} ${architectural_calibrations['joint_4']['yaw']}" />
       <parent
         link="half_arm_2_link${prefix}" />
@@ -291,5 +312,7 @@
         name="joint_5${prefix}"
         type="revolute">
-        <origin xyz="0 -0.20843 -0.006375" rpy="-1.5708 2.2204E-16 -6.373E-17" />
+        <origin
+          xyz="${architectural_calibrations['joint_5']['x']} ${architectural_calibrations['joint_5']['y'] - 0.20843} ${architectural_calibrations['joint_5']['z'] - 0.006375}"
+          rpy="${architectural_calibrations['joint_5']['roll'] - PI/2} ${architectural_calibrations['joint_5']['pitch']} ${architectural_calibrations['joint_5']['yaw']}" />
         <parent
           link="forearm_link${prefix}" />
@@ -309,5 +332,7 @@
         name="joint_5${prefix}"
         type="continuous">
-        <origin xyz="0 -0.20843 -0.006375" rpy="-1.5708 2.2204E-16 -6.373E-17" />
+        <origin
+          xyz="${architectural_calibrations['joint_5']['x']} ${architectural_calibrations['joint_5']['y'] - 0.20843} ${architectural_calibrations['joint_5']['z'] - 0.006375}"
+          rpy="${architectural_calibrations['joint_5']['roll'] - PI/2} ${architectural_calibrations['joint_5']['pitch']} ${architectural_calibrations['joint_5']['yaw']}" />
         <parent
           link="forearm_link${prefix}" />
@@ -346,5 +371,7 @@
       name="joint_6${prefix}"
       type="revolute">
-      <origin xyz="0 0.00017505 -0.10593" rpy="1.5708 9.2076E-28 -8.2157E-15" />
+      <origin
+        xyz="${architectural_calibrations['joint_6']['x']} ${architectural_calibrations['joint_6']['y'] + 0.00017505} ${architectural_calibrations['joint_6']['z'] - 0.10593}"
+        rpy="${architectural_calibrations['joint_6']['roll'] + PI/2} ${architectural_calibrations['joint_6']['pitch']} ${architectural_calibrations['joint_6']['yaw']}" />
       <parent
         link="spherical_wrist_1_link${prefix}" />
@@ -407,5 +434,7 @@
         name="joint_7${prefix}"
         type="revolute">
-        <origin xyz="0 -0.10593 -0.00017505" rpy="-1.5708 -5.5511E-17 9.6396E-17" />
+        <origin
+          xyz="${architectural_calibrations['joint_7']['x']} ${architectural_calibrations['joint_7']['y'] - 0.10593} ${architectural_calibrations['joint_7']['z'] - 0.00017505}"
+          rpy="${architectural_calibrations['joint_7']['roll'] - PI/2} ${architectural_calibrations['joint_7']['pitch']} ${architectural_calibrations['joint_7']['yaw']}" />
         <parent
           link="spherical_wrist_2_link${prefix}" />
@@ -425,5 +454,7 @@
         name="joint_7${prefix}"
         type="continuous">
-        <origin xyz="0 -0.10593 -0.00017505" rpy="-1.5708 -5.5511E-17 9.6396E-17" />
+        <origin
+          xyz="${architectural_calibrations['joint_7']['x']} ${architectural_calibrations['joint_7']['y'] - 0.10593} ${architectural_calibrations['joint_7']['z'] - 0.00017505}"
+          rpy="${architectural_calibrations['joint_7']['roll'] - PI/2} ${architectural_calibrations['joint_7']['pitch']} ${architectural_calibrations['joint_7']['yaw']}" />
         <parent
           link="spherical_wrist_2_link${prefix}" />

File: kortex_description/robots/kortex_robot.xacro (robot description, xacro)
@@ -28,4 +28,14 @@
     use_external_cable:=false
     initial_positions:=${dict(joint_1=0.0,joint_2=0.0,joint_3=0.0,joint_4=0.0,joint_5=0.0,joint_6=0.0,joint_7=0.0)}
+    architectural_calibrations:=${
+    dict(
+      joint_1=dict(x=0, y=0, z=0, roll=0, pitch=0, yaw=0),
+      joint_2=dict(x=0, y=0, z=0, roll=0, pitch=0, yaw=0),
+      joint_3=dict(x=0, y=0, z=0, roll=0, pitch=0, yaw=0),
+      joint_4=dict(x=0, y=0, z=0, roll=0, pitch=0, yaw=0),
+      joint_5=dict(x=0, y=0, z=0, roll=0, pitch=0, yaw=0),
+      joint_6=dict(x=0, y=0, z=0, roll=0, pitch=0, yaw=0),
+      joint_7=dict(x=0, y=0, z=0, roll=0, pitch=0, yaw=0)
+    )}
     gripper_max_velocity:=100.0
     gripper_max_force:=100.0
@@ -59,5 +69,6 @@
       gripper_max_force="${gripper_max_force}"
       use_external_cable="${use_external_cable}"
-      initial_positions="${initial_positions}">
+      initial_positions="${initial_positions}"
+      architectural_calibrations="${architectural_calibrations}">
       <xacro:insert_block name="origin" />
     </xacro:load_arm>
